Commit message: visualize the robot in gazebo

File: src/panda_description/urdf/hand.xacro (robot description, xacro)
@@ -9,4 +9,5 @@
       </joint>
     </xacro:unless>
+    <!-- Hand Link -->
     <link name="${ns}_hand">
       <visual>
@@ -20,5 +21,11 @@
         </geometry>
       </collision>
+      <inertial>
+        <origin xyz="0 0 0" rpy="0 0 0"/>
+        <mass value="0.68"/>
+        <inertia ixx="0.1" ixy="0.0" ixz="0.0" iyy="0.1" iyz="0.0" izz="0.1"/>
+      </inertial>
     </link>
+    <!-- Left Finger Link -->
     <link name="${ns}_leftfinger">
       <visual>
@@ -32,5 +39,11 @@
         </geometry>
       </collision>
+      <inertial>
+        <origin xyz="0 0 0" rpy="0 0 0"/>
+        <mass value="0.01"/>
+        <inertia ixx="0.1" ixy="0.0" ixz="0.0" iyy="0.1" iyz="0.0" izz="0.1"/>
+      </inertial>
     </link>
+    <!-- Right Finger Link -->
     <link name="${ns}_rightfinger">
       <visual>
@@ -46,5 +59,11 @@
         </geometry>
       </collision>
+      <inertial>
+        <origin xyz="0 0 0" rpy="0 0 0"/>
+        <mass value="0.01"/>
+        <inertia ixx="0.1" ixy="0.0" ixz="0.0" iyy="0.1" iyz="0.0" izz="0.1"/>
+      </inertial>
     </link>
+    <!-- Joint from Hand to Left Finger -->
     <joint name="${ns}_finger_joint1" type="prismatic">
       <parent link="${ns}_hand"/>
@@ -54,4 +73,5 @@
       <limit effort="20" lower="0.0" upper="0.04" velocity="0.2"/>
     </joint>
+    <!-- Joint from Hand to Right Finger -->
     <joint name="${ns}_finger_joint2" type="prismatic">
       <parent link="${ns}_hand"/>

File: src/panda_description/urdf/panda_arm.urdf.xacro (robot description, xacro)
@@ -1,5 +1,5 @@
 <?xml version='1.0' encoding='utf-8'?>
 <robot xmlns:xacro="http://www.ros.org/wiki/xacro" name="panda">
-  <xacro:include filename="$(find panda_description)/robots/panda_arm.xacro" />
+  <xacro:include filename="$(find panda_description)/urdf/panda_arm.xacro" />
   <xacro:panda_arm />
 </robot>

File: src/panda_description/urdf/panda_arm.xacro (robot description, xacro)
@@ -9,4 +9,14 @@
       </joint>
     </xacro:unless>
+    <!-- Define constants -->
+    <xacro:property name="joint_damping" value="1.0"/>
+    <!-- Used for fixing robot to Gazebo 'base_link' -->
+    <link name="world"/>
+    <joint name="robot_to_world" type="fixed">
+      <parent link="world"/>
+      <child link="${arm_id}_link0"/>
+      <!-- <origin xyz="0.0 0.0 0.0" rpy="0.0 0.0 0.0" /> -->
+    </joint>
+    <!-- Link 0 -->
     <link name="${arm_id}_link0">
       <visual>
@@ -20,19 +30,13 @@
         </geometry>
       </collision>
-    </link>
-    <link name="${arm_id}_link1">
-      <visual>
-        <geometry>
-          <mesh filename="package://${description_pkg}/meshes/visual/link1.dae"/>
-        </geometry>
-      </visual>
-      <collision>
-        <geometry>
-          <mesh filename="package://${description_pkg}/meshes/collision/link1.stl"/>
-        </geometry>
-      </collision>
-    </link>
+      <inertial>
+        <origin xyz="0 0 0" rpy="0 0 0"/>
+        <mass value="3.06"/>
+        <inertia ixx="0.3" ixy="0.0" ixz="0.0" iyy="0.3" iyz="0.0" izz="0.3"/>
+      </inertial>
+    </link>
+    <!-- Joint to connect Link 0 and Link 1 -->
     <joint name="${arm_id}_joint1" type="revolute">
-      <safety_controller k_position="100.0" k_velocity="40.0" soft_lower_limit="-2.8973" soft_upper_limit="2.8973"/>
+      <!-- <safety_controller k_position="100.0" k_velocity="40.0" soft_lower_limit="-2.8973" soft_upper_limit="2.8973"/> -->
       <origin rpy="0 0 0" xyz="0 0 0.333"/>
       <parent link="${arm_id}_link0"/>
@@ -40,19 +44,27 @@
       <axis xyz="0 0 1"/>
       <limit effort="87" lower="-2.8973" upper="2.8973" velocity="2.1750"/>
-    </joint>
-    <link name="${arm_id}_link2">
-      <visual>
-        <geometry>
-          <mesh filename="package://${description_pkg}/meshes/visual/link2.dae"/>
-        </geometry>
-      </visual>
-      <collision>
-        <geometry>
-          <mesh filename="package://${description_pkg}/meshes/collision/link2.stl"/>
-        </geometry>
-      </collision>
-    </link>
+      <dynamics damping="${joint_damping}"/>
+    </joint>
+    <!-- Link 1 -->
+    <link name="${arm_id}_link1">
+      <visual>
+        <geometry>
+          <mesh filename="package://${description_pkg}/meshes/visual/link1.dae"/>
+        </geometry>
+      </visual>
+      <collision>
+        <geometry>
+          <mesh filename="package://${description_pkg}/meshes/collision/link1.stl"/>
+        </geometry>
+      </collision>
+      <inertial>
+        <origin xyz="0 0 0" rpy="0 0 0"/>
+        <mass value="2.34"/>
+        <inertia ixx="0.3" ixy="0.0" ixz="0.0" iyy="0.3" iyz="0.0" izz="0.3"/>
+      </inertial>
+    </link>
+    <!-- Joint to connect Link 1 and Link 2 -->
     <joint name="${arm_id}_joint2" type="revolute">
-      <safety_controller k_position="100.0" k_velocity="40.0" soft_lower_limit="-1.7628" soft_upper_limit="1.7628"/>
+      <!-- <safety_controller k_position="100.0" k_velocity="40.0" soft_lower_limit="-1.7628" soft_upper_limit="1.7628"/> -->
       <origin rpy="${-pi/2} 0 0" xyz="0 0 0"/>
       <parent link="${arm_id}_link1"/>
@@ -60,17 +72,25 @@
       <axis xyz="0 0 1"/>
       <limit effort="87" lower="-1.7628" upper="1.7628" velocity="2.1750"/>
-    </joint>
-    <link name="${arm_id}_link3">
-      <visual>
-        <geometry>
-          <mesh filename="package://${description_pkg}/meshes/visual/link3.dae"/>
-        </geometry>
-      </visual>
-      <collision>
-        <geometry>
-          <mesh filename="package://${description_pkg}/meshes/collision/link3.stl"/>
-        </geometry>
-      </collision>
-    </link>
+      <dynamics damping="${joint_damping}"/>
+    </joint>
+    <!-- Link 2 -->
+    <link name="${arm_id}_link2">
+      <visual>
+        <geometry>
+          <mesh filename="package://${description_pkg}/meshes/visual/link2.dae"/>
+        </geometry>
+      </visual>
+      <collision>
+        <geometry>
+          <mesh filename="package://${description_pkg}/meshes/collision/link2.stl"/>
+        </geometry>
+      </collision>
+      <inertial>
+        <origin xyz="0 0 0" rpy="0 0 0"/>
+        <mass value="2.36"/>
+        <inertia ixx="0.3" ixy="0.0" ixz="0.0" iyy="0.3" iyz="0.0" izz="0.3"/>
+      </inertial>
+    </link>
+    <!-- Joint to connect Link 2 and Link 3 -->
     <joint name="${arm_id}_joint3" type="revolute">
       <safety_controller k_position="100.0" k_velocity="40.0" soft_lower_limit="-2.8973" soft_upper_limit="2.8973"/>
@@ -80,17 +100,25 @@
       <axis xyz="0 0 1"/>
       <limit effort="87" lower="-2.8973" upper="2.8973" velocity="2.1750"/>
-    </joint>
-    <link name="${arm_id}_link4">
-      <visual>
-        <geometry>
-          <mesh filename="package://${description_pkg}/meshes/visual/link4.dae"/>
-        </geometry>
-      </visual>
-      <collision>
-        <geometry>
-          <mesh filename="package://${description_pkg}/meshes/collision/link4.stl"/>
-        </geometry>
-      </collision>
-    </link>
+      <dynamics damping="${joint_damping}"/>
+    </joint>
+    <!-- Link 3 -->
+    <link name="${arm_id}_link3">
+      <visual>
+        <geometry>
+          <mesh filename="package://${description_pkg}/meshes/visual/link3.dae"/>
+        </geometry>
+      </visual>
+      <collision>
+        <geometry>
+          <mesh filename="package://${description_pkg}/meshes/collision/link3.stl"/>
+        </geometry>
+      </collision>
+      <inertial>
+        <origin xyz="0 0 0" rpy="0 0 0"/>
+        <mass value="2.38"/>
+        <inertia ixx="0.3" ixy="0.0" ixz="0.0" iyy="0.3" iyz="0.0" izz="0.3"/>
+      </inertial>
+    </link>
+    <!-- Joint to connect Link 3 and Link 4 -->
     <joint name="${arm_id}_joint4" type="revolute">
       <safety_controller k_position="100.0" k_velocity="40.0" soft_lower_limit="-3.0718" soft_upper_limit="-0.0698"/>
@@ -100,17 +128,25 @@
       <axis xyz="0 0 1"/>
       <limit effort="87" lower="-3.0718" upper="-0.0698" velocity="2.1750"/>
-    </joint>
-    <link name="${arm_id}_link5">
-      <visual>
-        <geometry>
-          <mesh filename="package://${description_pkg}/meshes/visual/link5.dae"/>
-        </geometry>
-      </visual>
-      <collision>
-        <geometry>
-          <mesh filename="package://${description_pkg}/meshes/collision/link5.stl"/>
-        </geometry>
-      </collision>
-    </link>
+      <dynamics damping="${joint_damping}"/>
+    </joint>
+    <!-- Link 4 -->
+    <link name="${arm_id}_link4">
+      <visual>
+        <geometry>
+          <mesh filename="package://${description_pkg}/meshes/visual/link4.dae"/>
+        </geometry>
+      </visual>
+      <collision>
+        <geometry>
+          <mesh filename="package://${description_pkg}/meshes/collision/link4.stl"/>
+        </geometry>
+      </collision>
+      <inertial>
+        <origin xyz="0 0 0" rpy="0 0 0"/>
+        <mass value="2.43"/>
+        <inertia ixx="0.3" ixy="0.0" ixz="0.0" iyy="0.3" iyz="0.0" izz="0.3"/>
+      </inertial>
+    </link>
+    <!-- Joint to connect Link 4 and Link 5 -->
     <joint name="${arm_id}_joint5" type="revolute">
       <safety_controller k_position="100.0" k_velocity="40.0" soft_lower_limit="-2.8973" soft_upper_limit="2.8973"/>
@@ -120,17 +156,25 @@
       <axis xyz="0 0 1"/>
       <limit effort="12" lower="-2.8973" upper="2.8973" velocity="2.6100"/>
-    </joint>
-    <link name="${arm_id}_link6">
-      <visual>
-        <geometry>
-          <mesh filename="package://${description_pkg}/meshes/visual/link6.dae"/>
-        </geometry>
-      </visual>
-      <collision>
-        <geometry>
-          <mesh filename="package://${description_pkg}/meshes/collision/link6.stl"/>
-        </geometry>
-      </collision>
-    </link>
+      <dynamics damping="${joint_damping}"/>
+    </joint>
+    <!-- Link 5 -->
+    <link name="${arm_id}_link5">
+      <visual>
+        <geometry>
+          <mesh filename="package://${description_pkg}/meshes/visual/link5.dae"/>
+        </geometry>
+      </visual>
+      <collision>
+        <geometry>
+          <mesh filename="package://${description_pkg}/meshes/collision/link5.stl"/>
+        </geometry>
+      </collision>
+      <inertial>
+        <origin xyz="0 0 0" rpy="0 0 0"/>
+        <mass value="3.5"/>
+        <inertia ixx="0.3" ixy="0.0" ixz="0.0" iyy="0.3" iyz="0.0" izz="0.3"/>
+      </inertial>
+    </link>
+    <!-- Joint to connect Link 5 and Link 6 -->
     <joint name="${arm_id}_joint6" type="revolute">
       <safety_controller k_position="100.0" k_velocity="40.0" soft_lower_limit="-0.0175" soft_upper_limit="3.7525"/>
@@ -140,17 +184,25 @@
       <axis xyz="0 0 1"/>
       <limit effort="12" lower="-0.0175" upper="3.7525" velocity="2.6100"/>
-    </joint>
-    <link name="${arm_id}_link7">
-      <visual>
-        <geometry>
-          <mesh filename="package://${description_pkg}/meshes/visual/link7.dae"/>
-        </geometry>
-      </visual>
-      <collision>
-        <geometry>
-          <mesh filename="package://${description_pkg}/meshes/collision/link7.stl"/>
-        </geometry>
-      </collision>
-    </link>
+      <dynamics damping="${joint_damping}"/>
+    </joint>
+    <!-- Link 6 -->
+    <link name="${arm_id}_link6">
+      <visual>
+        <geometry>
+          <mesh filename="package://${description_pkg}/meshes/visual/link6.dae"/>
+        </geometry>
+      </visual>
+      <collision>
+        <geometry>
+          <mesh filename="package://${description_pkg}/meshes/collision/link6.stl"/>
+        </geometry>
+      </collision>
+      <inertial>
+        <origin xyz="0 0 0" rpy="0 0 0"/>
+        <mass value="1.47"/>
+        <inertia ixx="0.3" ixy="0.0" ixz="0.0" iyy="0.3" iyz="0.0" izz="0.3"/>
+      </inertial>
+    </link>
+    <!-- Joint to connect Link 6 and Link 7 -->
     <joint name="${arm_id}_joint7" type="revolute">
       <safety_controller k_position="100.0" k_velocity="40.0" soft_lower_limit="-2.8973" soft_upper_limit="2.8973"/>
@@ -160,6 +212,25 @@
       <axis xyz="0 0 1"/>
       <limit effort="12" lower="-2.8973" upper="2.8973" velocity="2.6100"/>
-    </joint>
-    <link name="${arm_id}_link8"/>
+      <dynamics damping="${joint_damping}"/>
+    </joint>
+    <!-- Link 7 -->
+    <link name="${arm_id}_link7">
+      <visual>
+        <geometry>
+          <mesh filename="package://${description_pkg}/meshes/visual/link7.dae"/>
+        </geometry>
+      </visual>
+      <collision>
+        <geometry>
+          <mesh filename="package://${description_pkg}/meshes/collision/link7.stl"/>
+        </geometry>
+      </collision>
+      <inertial>
+        <origin xyz="0 0 0" rpy="0 0 0"/>
+        <mass value="0.45"/>
+        <inertia ixx="0.3" ixy="0.0" ixz="0.0" iyy="0.3" iyz="0.0" izz="0.3"/>
+      </inertial>
+    </link>
+    <!-- Joint to connect Link 7 and Link 8 -->
     <joint name="${arm_id}_joint8" type="fixed">
       <origin rpy="0 0 0" xyz="0 0 0.107"/>
@@ -168,4 +239,12 @@
       <axis xyz="0 0 0"/>
     </joint>
+    <!-- Link 8 -->
+    <link name="${arm_id}_link8">
+    <inertial>
+        <origin xyz="0 0 0" rpy="0 0 0"/>
+        <mass value="0.0"/>
+        <inertia ixx="0.3" ixy="0.0" ixz="0.0" iyy="0.3" iyz="0.0" izz="0.3"/>
+      </inertial>
+    </link>
   </xacro:macro>
 </robot>

File: src/panda_description/urdf/panda_arm_hand.urdf.xacro (robot description, xacro)
@@ -1,7 +1,10 @@
 <?xml version="1.0" encoding="utf-8"?>
 <robot xmlns:xacro="http://www.ros.org/wiki/xacro" name="panda">
+  <xacro:arg name="robot_name" default="panda"/>
   <xacro:include filename="$(find panda_description)/urdf/panda_arm.xacro"/>
   <xacro:include filename="$(find panda_description)/urdf/hand.xacro"/>
+  <xacro:include filename="$(find panda_description)/urdf/panda.gazebo.xacro"/>
   <xacro:panda_arm />
   <xacro:hand ns="panda" rpy="0 0 ${-pi/4}" connected_to="panda_link8"/>
+  <xacro:panda_gazebo robot_name="$(arg robot_name)" />
 </robot>

Commit message: basic ros_control functionality for manipulator

File: src/panda_description/urdf/hand.xacro (robot description, xacro)
@@ -73,4 +73,15 @@
       <limit effort="20" lower="0.0" upper="0.04" velocity="0.2"/>
     </joint>
+    <!-- Transmission element for Joint from Hand to Left Finger -->
+    <transmission name="${ns}_leftfinger">
+      <type>transmission_interface/SimpleTransmission</type>
+      <joint name="${ns}_finger_joint1">
+        <hardwareInterface>hardware_interface/EffortJointInterface</hardwareInterface>
+      </joint>
+      <actuator name="${ns}_finger_joint1">
+        <hardwareInterface>hardware_interface/EffortJointInterface</hardwareInterface>
+        <mechanicalReduction>1</mechanicalReduction>
+      </actuator>
+    </transmission>
     <!-- Joint from Hand to Right Finger -->
     <joint name="${ns}_finger_joint2" type="prismatic">
@@ -82,4 +93,15 @@
       <mimic joint="${ns}_finger_joint1" />
     </joint>
+    <!-- Transmission element for Joint from Hand to Right Finger -->
+    <transmission name="${ns}_rightfinger">
+      <type>transmission_interface/SimpleTransmission</type>
+      <joint name="${ns}_finger_joint2">
+        <hardwareInterface>hardware_interface/EffortJointInterface</hardwareInterface>
+      </joint>
+      <actuator name="${ns}_finger_joint2">
+        <hardwareInterface>hardware_interface/EffortJointInterface</hardwareInterface>
+        <mechanicalReduction>1</mechanicalReduction>
+      </actuator>
+    </transmission>
   </xacro:macro>
 </robot>

File: src/panda_description/urdf/panda.gazebo.xacro (robot description, xacro)
@@ -3,5 +3,5 @@
     <xacro:macro name="panda_gazebo" params="robot_name">
         <!-- Load Gazebo lib and set the robot namespace -->
-        <!-- <gazebo>
+        <gazebo>
             <plugin name="gazebo_ros_control" filename="libgazebo_ros_control.so">
                 <robotNamespace>/${robot_name}</robotNamespace>
@@ -9,5 +9,5 @@
                 <legacyModeNS>true</legacyModeNS>
             </plugin>
-        </gazebo> -->
+        </gazebo>
         <!-- Link 0 -->
         <gazebo reference="${robot_name}_link0">

File: src/panda_description/urdf/panda_arm.xacro (robot description, xacro)
@@ -36,5 +36,5 @@
       </inertial>
     </link>
-    <!-- Joint to connect Link 0 and Link 1 -->
+    <!-- Joint 1 connects Link 0 and Link 1 -->
     <joint name="${arm_id}_joint1" type="revolute">
       <!-- <safety_controller k_position="100.0" k_velocity="40.0" soft_lower_limit="-2.8973" soft_upper_limit="2.8973"/> -->
@@ -46,4 +46,15 @@
       <dynamics damping="${joint_damping}"/>
     </joint>
+    <!-- Transmission element for Joint 1 -->
+    <transmission name="${arm_id}_tran_1">
+      <type>transmission_interface/SimpleTransmission</type>
+      <joint name="${arm_id}_joint1">
+        <hardwareInterface>hardware_interface/EffortJointInterface</hardwareInterface>
+      </joint>
+      <actuator name="${arm_id}_motor_1">
+        <hardwareInterface>hardware_interface/EffortJointInterface</hardwareInterface>
+        <mechanicalReduction>1</mechanicalReduction>
+      </actuator>
+    </transmission>
     <!-- Link 1 -->
     <link name="${arm_id}_link1">
@@ -64,5 +75,5 @@
       </inertial>
     </link>
-    <!-- Joint to connect Link 1 and Link 2 -->
+    <!-- Joint 2 connects Link 1 and Link 2 -->
     <joint name="${arm_id}_joint2" type="revolute">
       <!-- <safety_controller k_position="100.0" k_velocity="40.0" soft_lower_limit="-1.7628" soft_upper_limit="1.7628"/> -->
@@ -74,4 +85,15 @@
       <dynamics damping="${joint_damping}"/>
     </joint>
+    <!-- Transmission element for Joint 2 -->
+    <transmission name="${arm_id}_tran_2">
+      <type>transmission_interface/SimpleTransmission</type>
+      <joint name="${arm_id}_joint2">
+        <hardwareInterface>hardware_interface/EffortJointInterface</hardwareInterface>
+      </joint>
+      <actuator name="${arm_id}_motor_2">
+        <hardwareInterface>hardware_interface/EffortJointInterface</hardwareInterface>
+          <mechanicalReduction>1</mechanicalReduction>
+      </actuator>
+    </transmission>
     <!-- Link 2 -->
     <link name="${arm_id}_link2">
@@ -92,5 +114,5 @@
       </inertial>
     </link>
-    <!-- Joint to connect Link 2 and Link 3 -->
+    <!-- Joint 3 connects Link 2 and Link 3 -->
     <joint name="${arm_id}_joint3" type="revolute">
       <safety_controller k_position="100.0" k_velocity="40.0" soft_lower_limit="-2.8973" soft_upper_limit="2.8973"/>
@@ -102,4 +124,15 @@
       <dynamics damping="${joint_damping}"/>
     </joint>
+    <!-- Transmission element for Joint 3 -->
+    <transmission name="${arm_id}_tran_3">
+      <type>transmission_interface/SimpleTransmission</type>
+      <joint name="${arm_id}_joint3">
+        <hardwareInterface>hardware_interface/EffortJointInterface</hardwareInterface>
+      </joint>
+      <actuator name="${arm_id}_motor_3">
+        <hardwareInterface>hardware_interface/EffortJointInterface</hardwareInterface>
+        <mechanicalReduction>1</mechanicalReduction>
+      </actuator>
+    </transmission>
     <!-- Link 3 -->
     <link name="${arm_id}_link3">
@@ -120,5 +153,5 @@
       </inertial>
     </link>
-    <!-- Joint to connect Link 3 and Link 4 -->
+    <!-- Joint 4 connects Link 3 and Link 4 -->
     <joint name="${arm_id}_joint4" type="revolute">
       <safety_controller k_position="100.0" k_velocity="40.0" soft_lower_limit="-3.0718" soft_upper_limit="-0.0698"/>
@@ -130,4 +163,15 @@
       <dynamics damping="${joint_damping}"/>
     </joint>
+    <!-- Transmission element for Joint 4 -->
+    <transmission name="${arm_id}_tran_4">
+      <type>transmission_interface/SimpleTransmission</type>
+      <joint name="${arm_id}_joint4">
+        <hardwareInterface>hardware_interface/EffortJointInterface</hardwareInterface>
+      </joint>
+      <actuator name="${arm_id}_motor_4">
+        <hardwareInterface>hardware_interface/EffortJointInterface</hardwareInterface>
+        <mechanicalReduction>1</mechanicalReduction>
+      </actuator>
+    </transmission>
     <!-- Link 4 -->
     <link name="${arm_id}_link4">
@@ -148,5 +192,5 @@
       </inertial>
     </link>
-    <!-- Joint to connect Link 4 and Link 5 -->
+    <!-- Joint 5 connects Link 4 and Link 5 -->
     <joint name="${arm_id}_joint5" type="revolute">
       <safety_controller k_position="100.0" k_velocity="40.0" soft_lower_limit="-2.8973" soft_upper_limit="2.8973"/>
@@ -158,4 +202,15 @@
       <dynamics damping="${joint_damping}"/>
     </joint>
+    <!-- Transmission element for Joint 5 -->
+    <transmission name="${arm_id}_tran_5">
+      <type>transmission_interface/SimpleTransmission</type>
+      <joint name="${arm_id}_joint5">
+        <hardwareInterface>hardware_interface/EffortJointInterface</hardwareInterface>
+      </joint>
+      <actuator name="${arm_id}_motor_5">
+        <hardwareInterface>hardware_interface/EffortJointInterface</hardwareInterface>
+        <mechanicalReduction>1</mechanicalReduction>
+      </actuator>
+    </transmission>
     <!-- Link 5 -->
     <link name="${arm_id}_link5">
@@ -176,5 +231,5 @@
       </inertial>
     </link>
-    <!-- Joint to connect Link 5 and Link 6 -->
+    <!-- Joint 6 connects Link 5 and Link 6 -->
     <joint name="${arm_id}_joint6" type="revolute">
       <safety_controller k_position="100.0" k_velocity="40.0" soft_lower_limit="-0.0175" soft_upper_limit="3.7525"/>
@@ -186,4 +241,15 @@
       <dynamics damping="${joint_damping}"/>
     </joint>
+    <!-- Transmission element for Joint 6 -->
+    <transmission name="${arm_id}_tran_6">
+      <type>transmission_interface/SimpleTransmission</type>
+      <joint name="${arm_id}_joint6">
+        <hardwareInterface>hardware_interface/EffortJointInterface</hardwareInterface>
+      </joint>
+      <actuator name="${arm_id}_motor_6">
+        <hardwareInterface>hardware_interface/EffortJointInterface</hardwareInterface>
+        <mechanicalReduction>1</mechanicalReduction>
+      </actuator>
+    </transmission>
     <!-- Link 6 -->
     <link name="${arm_id}_link6">
@@ -204,5 +270,5 @@
       </inertial>
     </link>
-    <!-- Joint to connect Link 6 and Link 7 -->
+    <!-- Joint 7 connects Link 6 and Link 7 -->
     <joint name="${arm_id}_joint7" type="revolute">
       <safety_controller k_position="100.0" k_velocity="40.0" soft_lower_limit="-2.8973" soft_upper_limit="2.8973"/>
@@ -214,4 +280,15 @@
       <dynamics damping="${joint_damping}"/>
     </joint>
+    <!-- Transmission element for Joint 7 -->
+    <transmission name="${arm_id}_tran_7">
+      <type>transmission_interface/SimpleTransmission</type>
+      <joint name="${arm_id}_joint7">
+        <hardwareInterface>hardware_interface/EffortJointInterface</hardwareInterface>
+      </joint>
+      <actuator name="${arm_id}_motor_7">
+        <hardwareInterface>hardware_interface/EffortJointInterface</hardwareInterface>
+        <mechanicalReduction>1</mechanicalReduction>
+      </actuator>
+    </transmission>
     <!-- Link 7 -->
     <link name="${arm_id}_link7">
